File: AudioAmplifier/amplifier_schematics/analogCircuit.sch (KiCad schematic (older format))
At the start: 3 parts

Commit message: kicad
Parts:
- added R10, R11, R12, R17, R18, R7, R8, R9: 10K, Resistors_THT:R_Axial_DIN0207_L6.3mm_D2.5mm_P10.16mm_Horizontal, symbol R
- added R13, R14: 5K6, Resistors_THT:R_Axial_DIN0207_L6.3mm_D2.5mm_P10.16mm_Horizontal, symbol R
- added R15, R16: 3K6, Resistors_THT:R_Axial_DIN0207_L6.3mm_D2.5mm_P10.16mm_Horizontal, symbol R
- added R5, R6: 4K7, Resistors_THT:R_Axial_DIN0207_L6.3mm_D2.5mm_P10.16mm_Horizontal, symbol R
- added U5: MCP4161-103E/P, Don-Fet-driver:DIP254P762X533-8, symbol MCP4161-103E/P
- added U7: NE5532, Don-Fet-driver:DIP254P762X533-8, symbol NE5532
- added U8: OPA2134A, Don-Fet-driver:DIP254P762X533-8, symbol OPA2134A
- U4: renamed from U?; footprint DIP254P762X533-8 -> Don-Fet-driver:DIP254P762X533-8
- U6: renamed from U?; footprint (none) -> Don-Fet-driver:DIP254P762X533-8
Connections:
- net +12V: now also U7.8 (V+), U7.8 (V+), U8.8 (V+), U8.8 (V+)
- net +5V: now also U5.8 (VDD)
- net -12VA: now also U7.4 (V-), U7.4 (V-), U8.4 (V-), U8.4 (V-)
- net CS_0: now also U5.1 (~CS)
- net GND: now also U4.7 (P0B), U6.3 (+), U6.5 (+), U5.4 (VSS), U5.7 (P0B), U7.3 (+), U7.5 (+), U8.3 (+), U8.5 (+)
- net LEFT_IN: now also R5.2; no longer U6.3 (+)
- net MOSI: now also U5.3 (SDI/SDO)
- net RIGHT_IN: now also R6.2; no longer U6.5 (+)
- net SCK: now also U5.2 (SCK)
- net leftChannelBands/SIGNAL_IN: now reaches U6.1
- net leftChannelBands/SIGNAL_IN: now also U4.6 (P0W)
- net at U6.2 (-): now also U4.5 (P0A), R5.1
- net at U6.6 (-): now also R6.1, U5.5 (P0A)
- net rightChannelBands/SIGNAL_IN: now reaches U6.7
- net rightChannelBands/SIGNAL_IN: now also U5.6 (P0W)
- new net: R13.1, R7.1, R8.1, R9.1, U7.2 (-)
- new net: R13.2, R15.2, U7.1
- new net: R10.1, R11.1, R12.1, R14.1, U7.6 (-)
- new net: R14.2, R16.2, U7.7
- new net: R15.1, R17.1, U8.2 (-)
- new net: R16.1, R18.1, U8.6 (-)
- new net LEFT_OUT: R17.2, U8.1
- new net RIGHT_OUT: R18.2, U8.7
- new net leftChannelBands/SINGAL_HIGH: R9.2
- new net leftChannelBands/SINGAL_LOW: R7.2
- new net leftChannelBands/SINGAL_MID: R8.2
- new net rightChannelBands/SINGAL_HIGH: R12.2
- new net rightChannelBands/SINGAL_LOW: R10.2
- new net rightChannelBands/SINGAL_MID: R11.2
Other:
- note added: "LEFT CHANNEL"
- note added: "RIGHT CHANNEL"
- moved on the sheet: U4, U6B

Commit message: updated KICAD
Parts:
- added R33, R34: 100R, symbol R
Connections:
- net GND: no longer U4.7 (P0B), U5.7 (P0B)
- net at R5.1, U6.2 (-): now also R33.2; no longer U4.5 (P0A)
- net at R6.1, U6.6 (-): now also R34.2; no longer U5.5 (P0A)
- new net: R33.1, U4.5 (P0A)
- new net: R34.1, U5.5 (P0A)
- no-connect marks 0 -> 2
Changed lines of the file:
@@
 $EndComp
 $Comp
-L +12V #PWR020
+L +12V #PWR34
 U 1 1 58F9CD63
 P 6900 2600
-F 0 "#PWR020" H 6900 2450 50  0001 C CNN
+F 0 "#PWR34" H 6900 2450 50  0001 C CNN
 F 1 "+12V" H 6900 2740 50  0000 C CNN
 F 2 "" H 6900 2600 50  0000 C CNN
@@
 $EndComp
 $Comp
-L +12V #PWR021
+L +12V #PWR27
 U 1 1 58F9CD7D
 P 3100 3950
-F 0 "#PWR021" H 3100 3800 50  0001 C CNN
+F 0 "#PWR27" H 3100 3800 50  0001 C CNN
 F 1 "+12V" H 3100 4090 50  0000 C CNN
 F 2 "" H 3100 3950 50  0000 C CNN
@@
 $EndComp
 $Comp
-L -12VA #PWR022
+L -12VA #PWR29
 U 1 1 58F9CE3A
 P 3300 4750
-F 0 "#PWR022" H 3300 4600 50  0001 C CNN
+F 0 "#PWR29" H 3300 4600 50  0001 C CNN
 F 1 "-12VA" H 3300 4890 50  0000 C CNN
 F 2 "" H 3300 4750 50  0000 C CNN
@@
 $EndComp
 $Comp
-L -12VA #PWR023
+L -12VA #PWR28
 U 1 1 58F9CF27
 P 3300 2850
-F 0 "#PWR023" H 3300 2700 50  0001 C CNN
+F 0 "#PWR28" H 3300 2700 50  0001 C CNN
 F 1 "-12VA" H 3300 2990 50  0000 C CNN
 F 2 "" H 3300 2850 50  0000 C CNN
@@
 $EndComp
 $Comp
-L +5V #PWR024
+L +5V #PWR24
 U 1 1 58F9D059
 P 2800 1550
-F 0 "#PWR024" H 2800 1400 50  0001 C CNN
+F 0 "#PWR24" H 2800 1400 50  0001 C CNN
 F 1 "+5V" H 2800 1690 50  0000 C CNN
 F 2 "" H 2800 1550 50  0000 C CNN
@@
 $EndComp
 $Comp
-L GND #PWR025
+L GND #PWR20
 U 1 1 58F9D076
 P 1800 1950
-F 0 "#PWR025" H 1800 1700 50  0001 C CNN
+F 0 "#PWR20" H 1800 1700 50  0001 C CNN
 F 1 "GND" H 1800 1800 50  0000 C CNN
 F 2 "" H 1800 1950 50  0000 C CNN
@@
 $EndComp
 $Comp
-L GND #PWR026
+L GND #PWR22
 U 1 1 5909878B
 P 2450 2650
-F 0 "#PWR026" H 2450 2400 50  0001 C CNN
+F 0 "#PWR22" H 2450 2400 50  0001 C CNN
 F 1 "GND" H 2450 2500 50  0000 C CNN
 F 2 "" H 2450 2650 50  0000 C CNN
@@
 Wire Wire Line
 	3600 1800 3600 2400
-Wire Wire Line
-	2850 1900 2850 2500
 $Comp
 L MCP4161-103E/P U5
@@
 $EndComp
 $Comp
-L +5V #PWR027
+L +5V #PWR25
 U 1 1 59098C35
 P 2800 3450
-F 0 "#PWR027" H 2800 3300 50  0001 C CNN
+F 0 "#PWR25" H 2800 3300 50  0001 C CNN
 F 1 "+5V" H 2800 3590 50  0000 C CNN
 F 2 "" H 2800 3450 50  0000 C CNN
@@
 $EndComp
 $Comp
-L GND #PWR028
+L GND #PWR21
 U 1 1 59098C3B
 P 1800 3850
-F 0 "#PWR028" H 1800 3600 50  0001 C CNN
+F 0 "#PWR21" H 1800 3600 50  0001 C CNN
 F 1 "GND" H 1800 3700 50  0000 C CNN
 F 2 "" H 1800 3850 50  0000 C CNN
@@
 	2500 4400 2350 4400
 $Comp
-L GND #PWR029
+L GND #PWR23
 U 1 1 59098E37
 P 2450 4550
-F 0 "#PWR029" H 2450 4300 50  0001 C CNN
+F 0 "#PWR23" H 2450 4300 50  0001 C CNN
 F 1 "GND" H 2450 4400 50  0000 C CNN
 F 2 "" H 2450 4550 50  0000 C CNN
@@
 	3600 3700 3600 4300
 Connection ~ 3600 4300
-Wire Wire Line
-	2850 3800 2850 4400
 Connection ~ 2850 4400
 $Sheet
@@
 	6600 2850 6600 3150
 $Comp
-L GND #PWR030
+L GND #PWR32
 U 1 1 590A4F66
 P 6600 3150
-F 0 "#PWR030" H 6600 2900 50  0001 C CNN
+F 0 "#PWR32" H 6600 2900 50  0001 C CNN
 F 1 "GND" H 6600 3000 50  0000 C CNN
 F 2 "" H 6600 3150 50  0000 C CNN
@@
 	6400 3050 6700 3050
 $Comp
-L +12V #PWR031
+L +12V #PWR26
 U 1 1 590A52B6
 P 3100 2050
-F 0 "#PWR031" H 3100 1900 50  0001 C CNN
+F 0 "#PWR26" H 3100 1900 50  0001 C CNN
 F 1 "+12V" H 3100 2190 50  0000 C CNN
 F 2 "" H 3100 2050 50  0000 C CNN
@@
 	3100 2050 3100 2100
 $Comp
-L -12VA #PWR032
+L -12VA #PWR36
 U 1 1 590A533F
 P 7100 3400
-F 0 "#PWR032" H 7100 3250 50  0001 C CNN
+F 0 "#PWR36" H 7100 3250 50  0001 C CNN
 F 1 "-12VA" H 7100 3540 50  0000 C CNN
 F 2 "" H 7100 3400 50  0000 C CNN
@@
 	6900 3450 6900 3250
 $Comp
-L +12V #PWR033
+L +12V #PWR35
 U 1 1 590A56F0
 P 6900 4500
-F 0 "#PWR033" H 6900 4350 50  0001 C CNN
+F 0 "#PWR35" H 6900 4350 50  0001 C CNN
 F 1 "+12V" H 6900 4640 50  0000 C CNN
 F 2 "" H 6900 4500 50  0000 C CNN
@@
 	6600 4750 6600 5050
 $Comp
-L GND #PWR034
+L GND #PWR33
 U 1 1 590A5718
 P 6600 5050
-F 0 "#PWR034" H 6600 4800 50  0001 C CNN
+F 0 "#PWR33" H 6600 4800 50  0001 C CNN
 F 1 "GND" H 6600 4900 50  0000 C CNN
 F 2 "" H 6600 5050 50  0000 C CNN
@@
 	6400 4950 6700 4950
 $Comp
-L -12VA #PWR035
+L -12VA #PWR37
 U 1 1 590A571F
 P 7100 5300
-F 0 "#PWR035" H 7100 5150 50  0001 C CNN
+F 0 "#PWR37" H 7100 5150 50  0001 C CNN
 F 1 "-12VA" H 7100 5440 50  0000 C CNN
 F 2 "" H 7100 5300 50  0000 C CNN
@@
 	7600 2650 7600 3100
 $Comp
-L GND #PWR036
+L GND #PWR38
 U 1 1 590A715C
 P 7600 3100
-F 0 "#PWR036" H 7600 2850 50  0001 C CNN
+F 0 "#PWR38" H 7600 2850 50  0001 C CNN
 F 1 "GND" H 7600 2950 50  0000 C CNN
 F 2 "" H 7600 3100 50  0000 C CNN
@@
 	7600 4550 7600 5000
 $Comp
-L GND #PWR037
+L GND #PWR39
 U 1 1 590A724A
 P 7600 5000
-F 0 "#PWR037" H 7600 4750 50  0001 C CNN
+F 0 "#PWR39" H 7600 4750 50  0001 C CNN
 F 1 "GND" H 7600 4850 50  0000 C CNN
 F 2 "" H 7600 5000 50  0000 C CNN
@@
 $EndComp
 $Comp
-L -12VA #PWR038
+L -12VA #PWR43
 U 1 1 590A83DC
 P 8650 5200
-F 0 "#PWR038" H 8650 5050 50  0001 C CNN
+F 0 "#PWR43" H 8650 5050 50  0001 C CNN
 F 1 "-12VA" H 8650 5340 50  0000 C CNN
 F 2 "" H 8650 5200 50  0000 C CNN
@@
 	8450 5250 8450 5100
 $Comp
-L -12VA #PWR039
+L -12VA #PWR42
 U 1 1 590A8811
 P 8650 3300
-F 0 "#PWR039" H 8650 3150 50  0001 C CNN
+F 0 "#PWR42" H 8650 3150 50  0001 C CNN
 F 1 "-12VA" H 8650 3440 50  0000 C CNN
 F 2 "" H 8650 3300 50  0000 C CNN
@@
 	8450 3350 8450 3200
 $Comp
-L +12V #PWR040
+L +12V #PWR41
 U 1 1 590A898E
 P 8450 4250
-F 0 "#PWR040" H 8450 4100 50  0001 C CNN
+F 0 "#PWR41" H 8450 4100 50  0001 C CNN
 F 1 "+12V" H 8450 4390 50  0000 C CNN
 F 2 "" H 8450 4250 50  0000 C CNN
@@
 	8450 4250 8450 4300
 $Comp
-L +12V #PWR041
+L +12V #PWR40
 U 1 1 590A8BE7
 P 8450 2350
-F 0 "#PWR041" H 8450 2200 50  0001 C CNN
+F 0 "#PWR40" H 8450 2200 50  0001 C CNN
 F 1 "+12V" H 8450 2490 50  0000 C CNN
 F 2 "" H 8450 2350 50  0000 C CNN
@@
 RIGHT CHANNEL
 $Comp
-L GND #PWR042
-U 1 1 5918C1D2
-P 3350 1900
-F 0 "#PWR042" H 3350 1650 50  0001 C CNN
-F 1 "GND" H 3350 1750 50  0000 C CNN
-F 2 "" H 3350 1900 50  0000 C CNN
-F 3 "" H 3350 1900 50  0000 C CNN
-	1    3350 1900
-	1    0    0    -1
-$EndComp
-Wire Wire Line
-	3350 1900 3350 1700
-Wire Wire Line
-	3350 1700 2750 1700
-$Comp
-L GND #PWR043
-U 1 1 5918CB16
-P 3350 3800
-F 0 "#PWR043" H 3350 3550 50  0001 C CNN
-F 1 "GND" H 3350 3650 50  0000 C CNN
-F 2 "" H 3350 3800 50  0000 C CNN
-F 3 "" H 3350 3800 50  0000 C CNN
-	1    3350 3800
-	1    0    0    -1
-$EndComp
-Wire Wire Line
-	3350 3800 3350 3600
-Wire Wire Line
-	3350 3600 2750 3600
+L R R33
+U 1 1 592BE9D1
+P 2850 2100
+F 0 "R33" V 2930 2100 50  0000 C CNN
+F 1 "100R" V 2850 2100 50  0000 C CNN
+F 2 "" V 2780 2100 50  0000 C CNN
+F 3 "" H 2850 2100 50  0000 C CNN
+	1    2850 2100
+	1    0    0    -1
+$EndComp
+$Comp
+L R R34
+U 1 1 592BEB8F
+P 2850 4000
+F 0 "R34" V 2930 4000 50  0000 C CNN
+F 1 "100R" V 2850 4000 50  0000 C CNN
+F 2 "" V 2780 4000 50  0000 C CNN
+F 3 "" H 2850 4000 50  0000 C CNN
+	1    2850 4000
+	1    0    0    -1
+$EndComp
+Wire Wire Line
+	2850 1900 2850 1950
+Wire Wire Line
+	2850 2250 2850 2500
+Wire Wire Line
+	2850 3800 2850 3850
+Wire Wire Line
+	2850 4150 2850 4400
+NoConn ~ 2750 1700
+NoConn ~ 2750 3600
 $EndSCHEMATC
